File: schematics/mcu.kicad_sch (KiCad schematic)
At the start: 1 part, among them U2 STM32F103C8Tx

Commit message: 2. | 2026-02-23 | Mo
Parts:
- added C7: 100nF, Capacitor_SMD:C_0603_1608Metric, symbol Device:C
- added C9: 100nF, Capacitor_SMD:C_0805_2012Metric, symbol Device:C
- added R6: 2.2k, Resistor_SMD:R_0402_1005Metric, symbol Device:R
- added SW1: SW_Push, Button_Switch_SMD:SW_Push_1P1T-SH_NO_CK_KMR2xxG, symbol Switch:SW_Push
- added Y1: ECS-2520MV-xxx-xx, Oscillator:Oscillator_SMD_ECS_2520MV-xxx-xx-4Pin_2.5x2.0mm, symbol Oscillator:ECS-2520MV-xxx-xx
Connections:
- net +3.3V: now reaches U2.1 (VBAT)
- net +3.3V: now also U2.24 (VDD), U2.36 (VDD), U2.48 (VDD), U2.9 (VDDA), C7.1, C9.2, SW1.1, Y1.1 (Tri-State), Y1.4 (VDD)
- net GND: now reaches U2.23 (VSS), U2.35 (VSS), U2.47 (VSS)
- net GND: now also U2.8 (VSSA), C7.2, C9.1, R6.1, Y1.2 (GND)
- net I2C_scl_master: now reaches U2.29 (PA8)
- net I2C_sda_master: now reaches U2.30 (PA9)
- net at U2.7 (NRST): now also R6.2, SW1.2
- new net Clock_Out: Y1.3 (OUT)
- no-connect marks 0 -> 2
Other:
- note added: "Clock"
