File: schematics/mcu.kicad_sch (KiCad schematic)
At the start: 7 parts, among them SW1 SW_Push, U2 STM32F103C8Tx, Y1 ECS-2520MV-xxx-xx

Commit message: 2026-02-25 | Mi
Parts:
- added C10, C12, C13, C14: 100nF, Capacitor_SMD:C_0805_2012Metric, symbol Device:C
- added C11: 20pF, Capacitor_SMD:C_0805_2012Metric, symbol Device:C
- added R8: 10k, Resistor_SMD:R_0402_1005Metric, symbol Device:R
- R6: value 2.2k -> 100k
Connections:
- net +3.3V: now also C12.2, C13.2, C14.2
- net Clock_Out: now also U2.5 (PD0), C11.2
- net GND: now also C10.1, C11.1, C12.1, C13.1, C14.1, R8.1
- net I2C_scl_master: now also U2.42 (PB6); no longer U2.29 (PA8)
- net I2C_sda_master: now also U2.43 (PB7); no longer U2.30 (PA9)
- net at R6.2, SW1.2, U2.7 (NRST): now also C10.2
- net at U2.20 (PB2): now also R8.2
- no-connect marks 2 -> 5
Other:
- moved on the sheet: R6, R7

Commit message: 2026-02-26 | Do
Parts:
- added R9: 10k, Resistor_SMD:R_0402_1005Metric, symbol Device:R
- C11: value 20pF -> 100nF
- SW1: footprint Button_Switch_SMD:SW_Push_1P1T-SH_NO_CK_KMR2xxG -> Button_Switch_SMD:SW_Push_1P1T_NO_CK_KMR2
- Y1: footprint Oscillator:Oscillator_SMD_ECS_2520MV-xxx-xx-4Pin_2.5x2.0mm -> Oscillator:Oscillator_SMD_EuroQuartz_XO53-4Pin_5.0x3.2mm
Connections:
- net +3.3V: now also R9.1
- net SWDIO: now reaches U2.34 (PA13)
- net SWDIO: now also R9.2
- net SWCLK: now reaches U2.37 (PA14)
- net SPI_miso_master: no longer names the net of U2.16 (PA6)
- no-connect marks 5 -> 28
Other:
- moved on the sheet: C10, C11, C12, C13, C14, C9, R6, R7, R8

Commit message: 2026-02-28
Connections:
- net +3.3V: now also R9.2; no longer R9.1
- net SWDIO: now also R9.1; no longer R9.2
- no-connect marks 28 -> 27
Other:
- moved on the sheet: R9

Commit message: 2026-03-01 | 2
Parts:
- C10, C11, C12, C13, C14, C9: footprint Capacitor_SMD:C_0805_2012Metric -> Capacitor_SMD:C_0603_1608Metric
Connections:
- net SPI_dc_master: now reaches U2.10 (PA0)
- net SPI_rst_master: now reaches U2.11 (PA1)
- net SPI_nss_master renamed SPI_cs_master
- no-connect marks 27 -> 26
Other:
- moved on the sheet: C10, C11, C12, C13, C14, C9, R6, R7, R8, R9

Commit message: 2026-03-09 | So-Mo
Parts:
- removed C11: 100nF, Capacitor_SMD:C_0603_1608Metric, symbol Device:C
Connections:
- net +3.3V: now also R6.1; no longer SW1.1
- net GND: now also SW1.1; no longer R6.1

Commit message: 2026-03-11
Connections:
- net SPI_sck_master: now also U2.41 (PB5)
- net T0_out: now reaches U2.12 (PA2)
- net R0_in: now reaches U2.13 (PA3)
- no-connect marks 26 -> 23
Changed lines of the file:
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@@
 	)
 	(rectangle
-		(start 22.86 57.15)
-		(end 107.95 158.75)
+		(start 22.86 58.42)
+		(end 107.95 160.02)
 		(stroke
 			(width 0.2)
@@
 	)
 	(no_connect
-		(at 50.8 121.92)
-	)
-	(no_connect
 		(at 50.8 119.38)
 	)
@@
 	)
 	(no_connect
-		(at 86.36 88.9)
-	)
-	(no_connect
-		(at 86.36 86.36)
-	)
-	(no_connect
 		(at 86.36 119.38)
 	)
@@
 	(wire
 		(pts
+			(xy 49.53 121.92) (xy 50.8 121.92)
+		)
+		(stroke
+			(width 0)
+			(type default)
+		)
+	)
+	(wire
+		(pts
 			(xy 40.64 81.28) (xy 41.91 81.28)
 		)
@@
 	(wire
 		(pts
+			(xy 87.63 88.9) (xy 86.36 88.9)
+		)
+		(stroke
+			(width 0)
+			(type default)
+		)
+	)
+	(wire
+		(pts
 			(xy 48.26 81.28) (xy 50.8 81.28)
 		)
@@
 		(pts
 			(xy 48.26 63.5) (xy 48.26 69.85)
+		)
+		(stroke
+			(width 0)
+			(type default)
+		)
+	)
+	(wire
+		(pts
+			(xy 87.63 86.36) (xy 86.36 86.36)
 		)
 		(stroke
@@
 		)
 	)
+	(global_label "T0_out"
+		(shape input)
+		(at 87.63 86.36 0)
+		(fields_autoplaced yes)
+		(effects
+			(font
+				(size 1.27 1.27)
+			)
+			(justify left)
+		)
+		(property "Intersheetrefs" "${INTERSHEET_REFS}"
+			(at 96.7836 86.36 0)
+			(effects
+				(font
+					(size 1.27 1.27)
+				)
+				(justify left)
+				(hide yes)
+			)
+		)
+	)
 	(global_label "SWDIO"
 		(shape output)
@@
 		)
 	)
+	(global_label "SPI_sck_master"
+		(shape input)
+		(at 49.53 121.92 180)
+		(fields_autoplaced yes)
+		(effects
+			(font
+				(size 1.27 1.27)
+			)
+			(justify right)
+		)
+		(property "Intersheetrefs" "${INTERSHEET_REFS}"
+			(at 31.9096 121.92 0)
+			(effects
+				(font
+					(size 1.27 1.27)
+				)
+				(justify right)
+				(hide yes)
+			)
+		)
+	)
 	(global_label "I2C_sda_master"
 		(shape input)
@@
 			(effects
 				(font
+					(size 1.27 1.27)
+				)
+				(justify left)
+				(hide yes)
+			)
+		)
+	)
+	(global_label "R0_in"
+		(shape input)
+		(at 87.63 88.9 0)
+		(fields_autoplaced yes)
+		(effects
+			(font
+				(size 1.27 1.27)
+			)
+			(justify left)
+		)
+		(property "Intersheetrefs" "${INTERSHEET_REFS}"
+			(at 95.8161 88.9 0)
+			(effects
+				(font
