File: schematics/peripherals.kicad_sch (KiCad schematic)
At the start: 3 parts, among them U3 SHT31-DIS

Commit message: 2. | 2026-02-23 | Mo
Parts:
- C5: footprint (none) -> Capacitor_SMD:C_0603_1608Metric
- R3: footprint (none) -> Resistor_SMD:R_0402_1005Metric
Changed lines of the file:
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@@
 	)
 	(rectangle
-		(start 25.4 25.4)
-		(end 88.9 55.88)
+		(start 25.4 55.88)
+		(end 88.9 25.4)
 		(stroke
 			(width 0.2)
@@
 	(wire
 		(pts
+			(xy 58.42 48.26) (xy 60.96 48.26)
+		)
+		(stroke
+			(width 0)
+			(type default)
+		)
+	)
+	(wire
+		(pts
 			(xy 43.18 33.02) (xy 58.42 33.02)
 		)
@@
 	(wire
 		(pts
+			(xy 69.85 41.91) (xy 69.85 40.64)
+		)
+		(stroke
+			(width 0)
+			(type default)
+		)
+	)
+	(wire
+		(pts
 			(xy 38.1 48.26) (xy 45.72 48.26)
 		)
@@
 	(wire
 		(pts
+			(xy 69.85 40.64) (xy 68.58 40.64)
+		)
+		(stroke
+			(width 0)
+			(type default)
+		)
+	)
+	(wire
+		(pts
 			(xy 45.72 48.26) (xy 58.42 48.26)
 		)
@@
 	(wire
 		(pts
-			(xy 69.85 38.1) (xy 69.85 36.83)
-		)
-		(stroke
-			(width 0)
-			(type default)
-		)
-	)
-	(wire
-		(pts
-			(xy 69.85 40.64) (xy 69.85 41.91)
+			(xy 69.85 36.83) (xy 69.85 38.1)
 		)
 		(stroke
@@
 	(wire
 		(pts
-			(xy 68.58 40.64) (xy 69.85 40.64)
+			(xy 69.85 41.91) (xy 71.12 41.91)
 		)
 		(stroke
@@
 		(pts
 			(xy 38.1 33.02) (xy 43.18 33.02)
-		)
-		(stroke
-			(width 0)
-			(type default)
-		)
-	)
-	(wire
-		(pts
-			(xy 69.85 41.91) (xy 71.12 41.91)
 		)
 		(stroke
@@
 				)
 				(justify right)
+				(hide yes)
+			)
+		)
+	)
+	(global_label "Gnd"
+		(shape output)
+		(at 60.96 48.26 0)
+		(fields_autoplaced yes)
+		(effects
+			(font
+				(size 1.27 1.27)
+			)
+			(justify left)
+		)
+		(property "Intersheetrefs" "${INTERSHEET_REFS}"
+			(at 67.5132 48.26 0)
+			(effects
+				(font
+					(size 1.27 1.27)
+				)
+				(justify left)
 				(hide yes)
 			)
@@
 			)
 		)
-		(property "Footprint" ""
+		(property "Footprint" "Resistor_SMD:R_0402_1005Metric"
 			(at 41.402 36.83 90)
 			(effects
@@
 			)
 		)
-		(property "Footprint" ""
+		(property "Footprint" "Capacitor_SMD:C_0603_1608Metric"
 			(at 39.0652 44.45 0)
 			(effects

Commit message: 2026-02-25 | Mi
Changed lines of the file:
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@@
 	)
 	(rectangle
-		(start 25.4 55.88)
-		(end 88.9 25.4)
+		(start 25.4 25.4)
+		(end 88.9 55.88)
 		(stroke
 			(width 0.2)

Commit message: 2026-02-26 | Do
Parts:
- removed C5: 100nF, Capacitor_SMD:C_0603_1608Metric, symbol Device:C
- removed R3: 10k, Resistor_SMD:R_0402_1005Metric, symbol Device:R
- removed U3: SHT31-DIS, Sensor_Humidity:Sensirion_DFN-8-1EP_2.5x2.5mm_P0.5mm_EP1.1x1.7mm, symbol Sensor_Humidity:SHT31-DIS
Connections:
- no-connect marks 2 -> 0
Other:
- note removed: "Senosr"
