File: schematics/communication.kicad_sch (KiCad schematic)
At the start: 19 parts, among them J2 Conn_01x05_Pin, J3 Conn_01x02_Pin, J4 Conn_01x08_Pin, U3 SHT31-DIS

Commit message: 2026-03-16
Parts:
- H1, H2, H3, H4: now in the parts list
Changed lines of the file:
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@@
 		(unit 1)
 		(exclude_from_sim no)
-		(in_bom no)
+		(in_bom yes)
 		(on_board yes)
 		(dnp no)
@@
 		(unit 1)
 		(exclude_from_sim no)
-		(in_bom no)
+		(in_bom yes)
 		(on_board yes)
 		(dnp no)
@@
 		(unit 1)
 		(exclude_from_sim no)
-		(in_bom no)
+		(in_bom yes)
 		(on_board yes)
 		(dnp no)
@@
 		(unit 1)
 		(exclude_from_sim no)
-		(in_bom no)
-		(on_board yes)
-		(dnp no)
+		(in_bom yes)
+		(on_board yes)
+		(dnp no)
