File: Temp-Project.kicad_sch (KiCad schematic)
At the start: 0 parts

Commit message: 2. | 2026-02-23 | Mo
Other:
- sheet Peripherals renamed Additional
Changed lines of the file:
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@@
 			(color 255 255 194 1.0000)
 		)
-		(property "Sheetname" "Peripherals"
+		(property "Sheetname" "Additional"
 			(at 184.15 97.0784 0)
 			(effects

Commit message: 2026-02-26 | Do
Other:
- removed sheet Communication
- sheet Additional: file schematics/peripherals.kicad_sch -> schematics/communication.kicad_sch
Changed lines of the file:
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@@
 	(title_block
 		(title "Main Page | Root")
-		(date "2026-02-22")
+		(date "2026-02-26")
 		(rev "0.1")
 		(company "seesee010, see Github for more informations")
@@
 	)
 	(sheet
-		(at 99.06 97.79)
-		(size 12.7 10.16)
-		(exclude_from_sim no)
-		(in_bom yes)
-		(on_board yes)
-		(dnp no)
-		(stroke
-			(width 0.2)
-			(type solid)
-			(color 0 0 0 1)
-		)
-		(fill
-			(color 255 255 194 1.0000)
-		)
-		(property "Sheetname" "Communication"
-			(at 98.806 97.028 0)
-			(effects
-				(font
-					(size 1.27 1.27)
-				)
-				(justify left bottom)
-			)
-		)
-		(property "Sheetfile" "schematics/communication.kicad_sch"
-			(at 99.06 108.5346 0)
-			(effects
-				(font
-					(size 1.27 1.27)
-				)
-				(justify left top)
-				(hide yes)
-			)
-		)
-		(instances
-			(project "Temp-Project"
-				(path "/c936f4ed-9370-4c35-ba8e-26b0afd3f3bd"
-					(page "5")
-				)
-			)
-		)
-	)
-	(sheet
-		(at 184.15 97.79)
+		(at 113.03 100.33)
 		(size 12.7 10.16)
 		(exclude_from_sim no)
@@
 		)
 		(property "Sheetname" "Additional"
-			(at 184.15 97.0784 0)
+			(at 112.776 99.568 0)
 			(effects
 				(font
@@
 			)
 		)
-		(property "Sheetfile" "schematics/peripherals.kicad_sch"
-			(at 177.038 107.95 0)
+		(property "Sheetfile" "schematics/communication.kicad_sch"
+			(at 113.03 111.0746 0)
 			(effects
 				(font
@@
 	)
 	(sheet
-		(at 127 97.79)
+		(at 140.97 100.33)
 		(size 12.7 10.16)
 		(exclude_from_sim no)
@@
 		)
 		(property "Sheetname" "Power"
-			(at 127 97.0784 0)
+			(at 140.97 99.6184 0)
 			(effects
 				(font
@@
 		)
 		(property "Sheetfile" "schematics/power-regulation.kicad_sch"
-			(at 119.38 108.458 0)
+			(at 133.35 110.998 0)
 			(effects
 				(font
@@
 	)
 	(sheet
-		(at 157.48 97.79)
+		(at 171.45 100.33)
 		(size 12.7 10.16)
 		(exclude_from_sim no)
@@
 		)
 		(property "Sheetname" "MCU"
-			(at 157.48 97.0784 0)
+			(at 171.45 99.6184 0)
 			(effects
 				(font
@@
 		)
 		(property "Sheetfile" "schematics/mcu.kicad_sch"
-			(at 154.686 108.458 0)
+			(at 168.656 110.998 0)
 			(effects
 				(font
