File: Temp-Project.kicad_pcb (KiCad board)
At the start: 2 copper layers, 40 parts, among them J1 USB_C_Receptacle_PowerOnly_6P, J2 Conn_01x05_Pin, J3 Conn_01x10_Pin, SW1 SW_Push, U1 AMS1117-3.3, U2 STM32F103C8Tx, U3 SHT31-DIS, Y1 ECS-2520MV-xxx-xx

Commit message: change the pic to a newer version
Routing:
- net SWCLK: track 0.00 -> 10.8 mm, vias 0 -> 2
- net +3.3V: track 77.9 -> 82.5 mm
- removed copper zone on B.Cu, net GND
- removed copper zone on F.Cu, net GND
Changed lines of the file:
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@@
+	)
+	(segment
+		(start 124.714 125.92)
+		(end 122.687788 127.946212)
+		(width 0.2)
+		(layer "F.Cu")
+		(net 2)
 	)
 	(segment
@@
 	)
 	(segment
+		(start 122.687788 127.946212)
+		(end 121.42466 127.946212)
+		(width 0.2)
+		(layer "F.Cu")
+		(net 2)
+	)
+	(segment
 		(start 118.11 133.737194)
 		(end 121.055523 133.737194)
@@
 		(start 121.738966 133.053751)
 		(end 121.738966 131.681119)
+		(width 0.2)
+		(layer "F.Cu")
+		(net 2)
+	)
+	(segment
+		(start 121.42466 127.946212)
+		(end 121.041744 128.329128)
 		(width 0.2)
 		(layer "F.Cu")
@@
 		(layer "F.Cu")
 		(net 7)
+	)
+	(segment
+		(start 122.92796 124.92)
+		(end 122.506528 124.498568)
+		(width 0.2)
+		(layer "F.Cu")
+		(net 8)
+	)
+	(segment
+		(start 120.123847 120.046153)
+		(end 119.8725 120.2975)
+		(width 0.2)
+		(layer "F.Cu")
+		(net 8)
+	)
+	(segment
+		(start 124.714 124.92)
+		(end 122.92796 124.92)
+		(width 0.2)
+		(layer "F.Cu")
+		(net 8)
+	)
+	(segment
+		(start 120.380415 120.046153)
+		(end 120.123847 120.046153)
+		(width 0.2)
+		(layer "F.Cu")
+		(net 8)
+	)
+	(segment
+		(start 120.610215 120.275953)
+		(end 120.380415 120.046153)
+		(width 0.2)
+		(layer "F.Cu")
+		(net 8)
+	)
+	(segment
+		(start 120.610215 120.475467)
+		(end 120.610215 120.275953)
+		(width 0.2)
+		(layer "F.Cu")
+		(net 8)
+	)
+	(via
+		(at 122.506528 124.498568)
+		(size 0.6)
+		(drill 0.3)
+		(layers "F.Cu" "B.Cu")
+		(net 8)
+	)
+	(via micro
+		(at 120.610215 120.475467)
+		(size 0.3)
+		(drill 0.1)
+		(layers "F.Cu" "B.Cu")
+		(net 8)
+	)
+	(segment
+		(start 119.255114 123.517529)
+		(end 119.255114 121.830568)
+		(width 0.2)
+		(layer "B.Cu")
+		(net 8)
+	)
+	(segment
+		(start 122.506528 124.498568)
+		(end 120.236153 124.498568)
+		(width 0.2)
+		(layer "B.Cu")
+		(net 8)
+	)
+	(segment
+		(start 119.255114 121.830568)
+		(end 120.610215 120.475467)
+		(width 0.2)
+		(layer "B.Cu")
+		(net 8)
+	)
+	(segment
+		(start 120.236153 124.498568)
+		(end 119.255114 123.517529)
+		(width 0.2)
+		(layer "B.Cu")
+		(net 8)
 	)
 	(segment
@@
 		(net 48)
 	)
-	(zone
-		(net 1)
-		(net_name "GND")
-		(layers "F.Cu" "B.Cu")
-		(hatch full 0.5)
-		(connect_pads
-			(clearance 0.25)
-		)
-		(min_thickness 0.2)
-		(filled_areas_thickness no)
-		(fill yes
-			(thermal_gap 0.5)
-			(thermal_bridge_width 0.5)
-		)
-		(polygon
-			(pts
-				(xy 85.5 112.5) (xy 127.75 112.5) (xy 127.75 136) (xy 85.5 136)
-			)
-		)
-	)
 	(embedded_fonts no)

Commit message: 2026-03-09 | So-Mo
Parts:
- removed C11: 100nF, Capacitor_SMD:C_0603_1608Metric
- removed J3: Conn_01x10_Pin, Connector_PinHeader_1.00mm:PinHeader_1x10_P1.00mm_Vertical
- added J4: Conn_01x08_Pin, Connector_PinHeader_1.00mm:PinHeader_1x08_P1.00mm_Vertical, F.Cu at (112.3, 132.7)
- TP1: value 5V -> TestPoint
- TP2: value 3.3V -> TestPoint
- TP3: value Clock -> TestPoint
- TP4: value Gnd -> TestPoint
- moved C3 0.18 mm to (95.7, 129.5)
- moved C15 0.12 mm to (115.9, 134.7)
Connections:
- R6 pad 1: GND -> +3.3V
- SW1 pad 1: +3.3V -> GND
Routing:
- net Clock_Out: track 29.6 -> 10.5 mm, vias 4 -> 2
- net +3.3V: track 82.5 -> 75.4 mm
- net +5V: track 23.3 -> 18.1 mm
- net SPI_dc_master: track 10.4 -> 8.81 mm
- net Net-(U2-PB2): track 10.1 -> 11.1 mm, vias 2 -> 3
- net Net-(U2-NRST): track 13.9 -> 13.1 mm
- net GND: track 11.4 -> 12.1 mm, vias 0 -> 63
- net SPI_sck_master: track 4.78 -> 5.12 mm, vias 0 -> 2
- net SPI_mosi_master: track 3.99 -> 4.04 mm, vias 2 -> 0
- added copper zone on B.Cu, net GND
- added copper zone on F.Cu, net GND
Other:
- board outline added: 42.2 x 23.5 mm

Commit message: 2026-03-11
Parts:
- removed C15: 100nF, Capacitor_SMD:C_0603_1608Metric
- added J3: Conn_01x02_Pin, Connector_PinHeader_2.54mm:PinHeader_1x02_P2.54mm_Vertical, F.Cu at (107.5, 116.9)
- J2: footprint Connector_PinHeader_1.00mm:PinHeader_1x04_P1.00mm_Vertical -> Connector_PinHeader_2.54mm:PinHeader_1x05_P2.54mm_Vertical
- J4: footprint Connector_PinHeader_1.00mm:PinHeader_1x08_P1.00mm_Vertical -> Connector_PinHeader_2.54mm:PinHeader_1x08_P2.54mm_Vertical
- moved R8 6.79 mm to (118.5, 130.2), turned to 180 degrees
- moved J4 5.13 mm to (107.2, 133.2)
- moved C8 5.08 mm to (114.3, 130.6)
- moved H3 3.94 mm to (129.2, 133.4)
- moved H2 3.94 mm to (129.2, 115.0)
- moved J2 3.23 mm to (125.4, 129.1)
- moved C14 3.21 mm to (110.5, 123.9), turned to -90 degrees
- moved C12 1.16 mm to (122.8, 129.6), turned to -90 degrees
- moved R5 0.52 mm to (114.3, 115.0), turned to 135 degrees
- moved H4 0.45 mm to (88.1, 133.3)
- moved C6 0.27 mm to (113.6, 116.8)
Connections:
- U2 pad 12: unconnected-(U2-PA2-Pad12) -> T0_out
- U2 pad 13: unconnected-(U2-PA3-Pad13) -> R0_in
- U2 pad 41: unconnected-(U2-PB5-Pad41) -> SPI_sck_master
Routing:
- net R0_in: track 0.00 -> 17.4 mm, vias 0 -> 1
- net T0_out: track 0.00 -> 13.2 mm, vias 0 -> 1
- net +3.3V: track 75.4 -> 87.3 mm, vias 0 -> 2
- net Net-(U2-PB2): track 11.1 -> 1.68 mm, vias 3 -> 0
- net GND: track 12.1 -> 19.9 mm, vias 63 -> 36
- net Clock_Out: track 10.5 -> 17.0 mm
- net SPI_sck_master: track 5.12 -> 9.55 mm
- net SPI_rst_master: track 7.30 -> 10.8 mm, vias 0 -> 2
- net SPI_dc_master: track 8.81 -> 12.3 mm
- net SPI_cs_master: track 4.25 -> 7.62 mm, vias 0 -> 2
- net SWCLK: track 10.7 -> 11.7 mm
- net SWDIO: track 3.58 -> 4.62 mm
- net SPI_mosi_master: track 4.04 -> 4.97 mm
Other:
- board size 42.2 x 23.5 mm -> 46.2 x 23.5 mm
- board text added: "seesee010"

Commit message: 2026-03-16
Parts:
- moved C13 1.48 mm to (121.8, 118.2)
Routing:
- net +3.3V: track 87.3 -> 110.0 mm
- net GND: track 19.9 -> 30.2 mm, vias 36 -> 37
- net Net-(U2-NRST): track 13.1 -> 17.2 mm
